File: keyboard/pcbs/main.kicad_pcb (KiCad board)
At the start: 2 copper layers, 139.5 x 130.1 mm, 60 parts

Commit message: updates
Parts:
- removed Nice!View1: , lib:niceview_headers
- added DISP1: , nice!view, F.Cu at (108.0, -42.5)
- moved MCU1 64.5 mm to (113.5, -46.7)
Other:
- board size 139.5 x 130.1 mm -> 141 x 130.1 mm

Commit message: latest stuff
Connections:
- D1 pad 1: (no net) -> P14
- D10 pad 1: (no net) -> P13
- D11 pad 1: (no net) -> P12
- D12 pad 1: (no net) -> P11
- D13 pad 1: (no net) -> P14
- D14 pad 1: (no net) -> P13
- D15 pad 1: (no net) -> P12
- D16 pad 1: (no net) -> P11
- D17 pad 1: (no net) -> P14
- D18 pad 1: (no net) -> P13
- D19 pad 1: (no net) -> P12
- D2 pad 1: (no net) -> P13
- D20 pad 1: (no net) -> P11
- D21 pad 1: (no net) -> P14
- D22 pad 1: (no net) -> P13
- D23 pad 1: (no net) -> P12
- D24 pad 1: (no net) -> P11
- D25 pad 1: (no net) -> P13
- D3 pad 1: (no net) -> P12
- D4 pad 1: (no net) -> P11
- D5 pad 1: (no net) -> P14
- D6 pad 1: (no net) -> P13
- D7 pad 1: (no net) -> P12
- D8 pad 1: (no net) -> P11
- D9 pad 1: (no net) -> P14
- S1 pad 1: (no net) -> P21
- S10 pad 1: (no net) -> P19
- S11 pad 1: (no net) -> P19
- S12 pad 1: (no net) -> P19
- S13 pad 1: (no net) -> P18
- S14 pad 1: (no net) -> P18
- S15 pad 1: (no net) -> P18
- S16 pad 1: (no net) -> P18
- S17 pad 1: (no net) -> P17
- S18 pad 1: (no net) -> P17
- S19 pad 1: (no net) -> P17
- S2 pad 1: (no net) -> P21
- S20 pad 1: (no net) -> P17
- S21 pad 1: (no net) -> P16
- S22 pad 1: (no net) -> P16
- S23 pad 1: (no net) -> P16
- S24 pad 1: (no net) -> P16
- S25 pad 1: (no net) -> P15
- S3 pad 1: (no net) -> P21
- S4 pad 1: (no net) -> P21
- S5 pad 1: (no net) -> P20
- S6 pad 1: (no net) -> P20
- S7 pad 1: (no net) -> P20
- S8 pad 1: (no net) -> P20
- S9 pad 1: (no net) -> P19
Routing:
- net outer_bottom: track 122.1 -> 0.00 mm
- net P21: track 0.00 -> 122.1 mm
- net ring_home: track 0.00 -> 122.0 mm
- net middle_bottom: track 122.0 -> 0.00 mm
- net inner_top: track 50.9 -> 0.00 mm
- net inner_num: track 50.9 -> 0.00 mm
- net index_top: track 0.00 -> 50.9 mm
- net index_home: track 0.00 -> 50.9 mm
