File: test/pcbs/mock_footprints___pcbs_main.kicad_pcb (KiCad board)
At the start: 2 copper layers, 39 x 19 mm, 8 parts

Commit message: mainnumpad
Parts:
- removed the ? at (0.00, 0.00) (x4)
- added ? (x2): , anchor_test, F.Cu at (0.00, 0.00)
- added ? (x2): , arrobj_test, F.Cu at (0.00, 0.00)
Changed lines of the file:
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@@
   (page A3)
   (title_block
-    (title main)
-    (rev v1.0.0)
-    (company Unknown)
+    (title "main")
+    (rev "v1.0.0")
+    (company "Unknown")
   )
   (general
@@
       (outputdirectory ""))
   )
-            (net 0 "")
+  (net 0 "")
 (net 1 "P1")
 (net 2 "T4_1")
@@
 (fp_line (start 5 5) (end 7 5) (layer Dwgs.User) (width 0.05))
                 )
-            (gr_line (start -9.5 9.5) (end 9.5 9.5) (angle 90) (layer Edge.Cuts) (width 0.15))
+  (gr_line (start -9.5 9.5) (end 9.5 9.5) (angle 90) (layer Edge.Cuts) (width 0.15))
 (gr_line (start 9.5 9.5) (end 9.5 -9.5) (angle 90) (layer Edge.Cuts) (width 0.15))
 (gr_line (start 9.5 -9.5) (end -9.5 -9.5) (angle 90) (layer Edge.Cuts) (width 0.15))
